Commit message: MoveItパッケージの追加

File: model/lifter_mover.ros2_control.xacro (robot description, xacro)
@@ -1,5 +1,5 @@
 <?xml version="1.0"?>
 <robot xmlns:xacro="http://www.ros.org/wiki/xacro">
-  <xacro:macro name="noid_ros2_control" params="name driver_settings">
+  <xacro:macro name="lifter_mover_ros2_control" params="name driver_settings">
     <ros2_control name="${name}" type="system">
       <hardware>

File: model/lifter_mover.urdf.xacro (robot description, xacro)
@@ -25,4 +25,4 @@
        top_link="${lifter_top_link}" />
     <xacro:include filename="$(find lifter_mover)/model/lifter_mover.ros2_control.xacro" />
-    <xacro:noid_ros2_control name="lifter_mover" driver_settings="$(arg driver_settings)" />
+    <xacro:lifter_mover_ros2_control name="lifter_mover" driver_settings="$(arg driver_settings)" />
 </robot>

File: model/lifter_mover_gz.urdf.xacro (robot description, xacro)
@@ -25,4 +25,4 @@
        top_link="${lifter_top_link}" />
     <xacro:include filename="$(find lifter_mover)/model/lifter_mover.ros2_control.xacro" />
-    <xacro:noid_ros2_control name="lifter_mover" driver_settings="$(arg driver_settings)" />
+    <xacro:lifter_mover_ros2_control name="lifter_mover" driver_settings="$(arg driver_settings)" />
 </robot>
